File: Arduino/schematic/mainboard/scrump.brd (EAGLE design)
At the start: 100 x 80 mm, 29 parts, among them J1 PINHEAD-FTSH, J2 USB-CON-5PIN-105017-0001, U1 ATSAMD21G-A, U2 LM3671, U3 MCP73831, Y1 32.768kHz

Commit message: Initial PCB
Parts:
- added D3: MBRA140, SparkFun-DiscreteSemi:SMA-DIODE
- added D4: RED 1.8V, SparkFun-LED:LED-0603
- C12: value 10uF -> 4.7uF
- C13: value 0.1uF -> 10uF
- C5: value 0.1uF -> 22pF
- C7: value 22pF -> 0.1uF
- C9: value 4.7uF -> 0.1uF
- D2: value RED 1.8V -> MBRA140; device SparkFun-LED:LED-0603 -> SparkFun-DiscreteSemi:SMA-DIODE
- L1: value 2.2uF -> 2.2uH
- R1: value 22R -> 330R
- R2: value 330R -> 1.5k
- R3: value 1.5k -> 5k
- R4: value 2k -> 22R
- moved J2 73.1 mm to (52.5, 75.8), turned to 180 degrees
- moved R2 64.8 mm to (59.9, 52.3), turned to 90 degrees
- moved C11 59.4 mm to (53.0, 62.0)
- moved C7 57.7 mm to (32.5, 56.5), turned to 90 degrees
- moved R1 57.5 mm to (35.5, 55.8), turned to 90 degrees
- moved C5 53.8 mm to (39.0, 46.2), turned to 180 degrees
- moved C12 50.6 mm to (56.0, 62.0)
- moved J1 50.1 mm to (38.0, 72.5), turned to 270 degrees
- moved C1 48.6 mm to (47.8, 47.2), turned to 180 degrees
- moved C8 48.2 mm to (49.2, 32.0), turned to 270 degrees
- moved C4 45.9 mm to (42.8, 39.2), turned to 270 degrees
- moved C3 45.4 mm to (50.8, 47.2)
- moved C10 45.4 mm to (57.2, 57.2), turned to 90 degrees
- moved U2 42.0 mm to (49.5, 52.8), turned to 180 degrees
- moved L1 40.9 mm to (49.5, 49.5)
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Connections:
- net PA02 renamed A0
- net PA03 renamed AREF
- net PA04 renamed A3
- net PA05 renamed A4
- net PA06 renamed D8
- net PA07 renamed D9
- net PA08 renamed D4
- net PA09 renamed D3
- net PA10 renamed D1
- net PA11 renamed D0
- net PA12 renamed MISO
- net PA14 renamed D2
- net PA15 renamed D5
- net PA16 renamed D11
- net PA17 renamed D13
- net PA18 renamed D10
- net PA19 renamed D12
- net PA20 renamed D6
- net PA21 renamed D7
- net PB02 renamed A5
- net PB08 renamed A1
- net PB09 renamed A2
- net PB10 renamed MOSI
- net PB11 renamed SCK
- net PB22 renamed TXD
- net PB23 renamed RXD
- removed net +5V: C11.1, D1.A, J2.1
- removed net PA00: C6.1, U1.1, Y1.P$1
- removed net PA01: C7.1, U1.2, Y1.P$4
- removed net VCC: C10.1, U2.1, U2.3, U3.3
- new net N$10: D2.C, D3.C, U2.1, U2.3
- new net V_BATT: C11.1, D3.A, U3.3
- new net V_USB: C12.1, D1.A, D2.A, J2.1
- new net XIN32: C5.1, U1.1, Y1.P$1
- new net XOUT32: C6.1, U1.2, Y1.P$4
- net +3V3: now also C8.1, C9.1; no longer C12.1, C5.1
- net D-: now also R4.2; no longer R1.2
- net GND: now also R3.1; no longer R4.1
- net N$2: now also R1.2; no longer R2.2
- net N$3: now also C10.1, R2.2; no longer C9.1, R3.2
- net N$6: now also D4.C; no longer D2.C
- net N$7: now also D4.A, R2.1; no longer D2.A, R3.1
- net N$8: now also R3.2; no longer R4.2
- net N$9: now also R4.1; no longer R1.1
- net RESET: now also C7.1, R1.1; no longer C8.1, R2.1
Routing:
- net +3V3: track 0.00 -> 44.3 mm
- net N$3: track 0.00 -> 17.6 mm, vias 0 -> 2
- net V_BATT: track 0.00 -> 10.1 mm
- net N$10: track 0.00 -> 9.92 mm
- net XOUT32: track 0.00 -> 9.11 mm
- net XIN32: track 0.00 -> 8.75 mm
- net D-: track 0.00 -> 4.11 mm
- net D+: track 0.00 -> 4.11 mm
- net N$6: track 0.00 -> 3.57 mm
- net N$1: track 0.00 -> 3.06 mm
- net N$5: track 0.00 -> 1.97 mm
- net V_USB: track 0.00 -> 1.77 mm
- net N$7: track 0.00 -> 1.46 mm
- net N$8: track 0.00 -> 1.32 mm
- added copper zone on layer 1, net GND

Commit message: PCB changes
Parts:
- moved B1 3.51 mm to (81.0, 49.5)
- moved C5 0.38 mm to (39.4, 46.2)
Changed lines of the file:
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@@
 </class>
 </classes>
-<designrules name="default">
+<designrules name="SeeedStudio_2layer_DRU_no_angle_20140221">
 <description language="de">&lt;b&gt;EAGLE Design Rules&lt;/b&gt;
 &lt;p&gt;
@@
 necessary adjustments and save your customized
 design rules under a new name.</description>
+<description language="zh">&lt;b&gt;Seeed Studio EAGLE Design Rules&lt;/b&gt;
+</description>
 <param name="layerSetup" value="(1*16)"/>
-<param name="mtCopper" value="0.035mm 0.035mm 0.035mm 0.035mm 0.035mm 0.035mm 0.035mm 0.035mm 0.035mm 0.035mm 0.035mm 0.035mm 0.035mm 0.035mm 0.035mm 0.035mm"/>
-<param name="mtIsolate" value="1.5mm 0.15mm 0.2mm 0.15mm 0.2mm 0.15mm 0.2mm 0.15mm 0.2mm 0.15mm 0.2mm 0.15mm 0.2mm 0.15mm 0.2mm"/>
-<param name="mdWireWire" value="8mil"/>
-<param name="mdWirePad" value="8mil"/>
-<param name="mdWireVia" value="8mil"/>
-<param name="mdPadPad" value="8mil"/>
-<param name="mdPadVia" value="8mil"/>
-<param name="mdViaVia" value="8mil"/>
-<param name="mdSmdPad" value="8mil"/>
-<param name="mdSmdVia" value="8mil"/>
-<param name="mdSmdSmd" value="8mil"/>
+<param name="mtCopper" value="0.035mm 0.0175mm 0.035mm 0.035mm 0.035mm 0.035mm 0.035mm 0.035mm 0.035mm 0.035mm 0.035mm 0.035mm 0.035mm 0.035mm 0.0175mm 0.035mm"/>
+<param name="mtIsolate" value="1.5mm 1.1mm 0.2mm 0.15mm 0.2mm 0.15mm 0.2mm 0.15mm 0.2mm 0.15mm 0.2mm 0.15mm 0.2mm 0.15mm 0.2mm"/>
+<param name="mdWireWire" value="6mil"/>
+<param name="mdWirePad" value="6mil"/>
+<param name="mdWireVia" value="6mil"/>
+<param name="mdPadPad" value="6mil"/>
+<param name="mdPadVia" value="6mil"/>
+<param name="mdViaVia" value="6mil"/>
+<param name="mdSmdPad" value="0mil"/>
+<param name="mdSmdVia" value="0mil"/>
+<param name="mdSmdSmd" value="0mil"/>
 <param name="mdViaViaSameLayer" value="8mil"/>
 <param name="mnLayersViaInSmd" value="2"/>
-<param name="mdCopperDimension" value="40mil"/>
-<param name="mdDrill" value="8mil"/>
+<param name="mdCopperDimension" value="10mil"/>
+<param name="mdDrill" value="10mil"/>
 <param name="mdSmdStop" value="0mil"/>
-<param name="msWidth" value="10mil"/>
-<param name="msDrill" value="24mil"/>
-<param name="msMicroVia" value="9.99mm"/>
+<param name="msWidth" value="6mil"/>
+<param name="msDrill" value="12mil"/>
+<param name="msMicroVia" value="12mil"/>
 <param name="msBlindViaRatio" value="0.5"/>
 <param name="rvPadTop" value="0.25"/>
@@
 <param name="rlMinPadBottom" value="10mil"/>
 <param name="rlMaxPadBottom" value="20mil"/>
-<param name="rlMinViaOuter" value="8mil"/>
+<param name="rlMinViaOuter" value="6mil"/>
 <param name="rlMaxViaOuter" value="20mil"/>
-<param name="rlMinViaInner" value="8mil"/>
+<param name="rlMinViaInner" value="6mil"/>
 <param name="rlMaxViaInner" value="20mil"/>
 <param name="rlMinMicroViaOuter" value="4mil"/>
@@
 <param name="psTop" value="-1"/>
 <param name="psBottom" value="-1"/>
-<param name="psFirst" value="-1"/>
+<param name="psFirst" value="0"/>
 <param name="psElongationLong" value="100"/>
 <param name="psElongationOffset" value="100"/>
 <param name="mvStopFrame" value="1"/>
 <param name="mvCreamFrame" value="0"/>
-<param name="mlMinStopFrame" value="4mil"/>
-<param name="mlMaxStopFrame" value="4mil"/>
+<param name="mlMinStopFrame" value="2mil"/>
+<param name="mlMaxStopFrame" value="2mil"/>
 <param name="mlMinCreamFrame" value="0mil"/>
 <param name="mlMaxCreamFrame" value="0mil"/>
-<param name="mlViaStopLimit" value="0mil"/>
+<param name="mlViaStopLimit" value="100mil"/>
 <param name="srRoundness" value="0"/>
 <param name="srMinRoundness" value="0mil"/>
@@
 <param name="checkAngle" value="0"/>
 <param name="checkFont" value="1"/>
-<param name="checkRestrict" value="1"/>
+<param name="checkRestrict" value="0"/>
 <param name="useDiameter" value="13"/>
 <param name="maxErrors" value="50"/>
@@
 <element name="Y1" library="mylibrary" package="ABS25" value="32.768kHz" x="37" y="42.5" rot="R180"/>
 <element name="C6" library="SparkFun-Capacitors" package="0603-CAP" value="22pF" x="39.375" y="39" rot="R180"/>
-<element name="C5" library="SparkFun-Capacitors" package="0603-CAP" value="22pF" x="39" y="46.25" rot="R180"/>
+<element name="C5" library="SparkFun-Capacitors" package="0603-CAP" value="22pF" x="39.375" y="46.25" rot="R180"/>
 <element name="U2" library="mylibrary" package="SOT23-5" value="LM3671" x="49.5" y="52.75" rot="R180"/>
 <element name="C13" library="SparkFun-Capacitors" package="0603-CAP" value="10uF" x="46.375" y="49.375" rot="R180"/>
@@
 <element name="R4" library="SparkFun-Resistors" package="0603-RES" value="22R" x="59" y="40.75" rot="R180"/>
 <element name="R5" library="SparkFun-Resistors" package="0603-RES" value="22R" x="59" y="42.25" rot="R180"/>
-<element name="B1" library="mylibrary" package="BMP180_BREAKOUT" value="BMP180BREAKOUT" x="84.5" y="49.25" rot="R270"/>
+<element name="B1" library="mylibrary" package="BMP180_BREAKOUT" value="BMP180BREAKOUT" x="81" y="49.5" rot="R270"/>
 <element name="D2" library="SparkFun-DiscreteSemi" package="SMA-DIODE" value="MBRA140" x="47.75" y="58.25" rot="R270">
 <attribute name="PROD_ID" value="DIO-08053" x="47.75" y="58.25" size="1.778" layer="27" rot="R270" display="off"/>
@@
 <wire x1="49.25" y1="43.25" x2="49.75" y2="42.75" width="0.3" layer="1"/>
 <wire x1="49.75" y1="42.75" x2="54.25" y2="42.75" width="0.3" layer="1"/>
-<wire x1="54.25" y1="44.65" x2="85.77" y2="44.17" width="0" layer="19" extent="1-1"/>
+<wire x1="54.25" y1="44.65" x2="82.27" y2="44.42" width="0" layer="19" extent="1-1"/>
 <wire x1="35.968" y1="75.04" x2="48.55" y2="51.4499" width="0" layer="19" extent="1-1"/>
 </signal>
@@
 <wire x1="39.75" y1="44.1" x2="41.1" y2="42.75" width="0.3" layer="1"/>
 <wire x1="41.1" y1="42.75" x2="45.75" y2="42.75" width="0.3" layer="1"/>
-<wire x1="39.85" y1="46.25" x2="39.75" y2="46.15" width="0.3" layer="1"/>
-<wire x1="39.75" y1="46.15" x2="39.75" y2="44.1" width="0.3" layer="1"/>
+<wire x1="40.225" y1="46.25" x2="39.75" y2="46.25" width="0.4064" layer="1"/>
+<wire x1="39.75" y1="46.25" x2="39.75" y2="44.1" width="0.4064" layer="1"/>
 </signal>
 <signal name="XOUT32">
@@
 <wire x1="39.75" y1="40.9" x2="41.1" y2="42.25" width="0.3" layer="1"/>
 <wire x1="41.1" y1="42.25" x2="45.75" y2="42.25" width="0.3" layer="1"/>
-<wire x1="40.225" y1="39" x2="39.75" y2="38.85" width="0.3" layer="1"/>
-<wire x1="39.75" y1="38.85" x2="39.75" y2="40.9" width="0.3" layer="1"/>
+<wire x1="40.225" y1="39" x2="39.75" y2="39" width="0.4064" layer="1"/>
+<wire x1="39.75" y1="39" x2="39.75" y2="40.9" width="0.4064" layer="1"/>
 </signal>
 <signal name="A0">
@@
 <contactref element="U1" pad="31"/>
 <contactref element="B1" pad="5"/>
-<wire x1="54.25" y1="40.25" x2="85.77" y2="36.55" width="0" layer="19" extent="1-1"/>
+<wire x1="54.25" y1="40.25" x2="82.27" y2="36.8" width="0" layer="19" extent="1-1"/>
 </signal>
 <signal name="SCL">
 <contactref element="U1" pad="32"/>
 <contactref element="B1" pad="4"/>
-<wire x1="54.25" y1="40.75" x2="85.77" y2="39.09" width="0" layer="19" extent="1-1"/>
+<wire x1="54.25" y1="40.75" x2="82.27" y2="39.34" width="0" layer="19" extent="1-1"/>
 </signal>
 <signal name="PA27">

Commit message: Added LDR
Parts:
- added B2: BMP180BREAKOUT, mylibrary:BMP180_BREAKOUT
- added R6: (no value), SparkFun-Resistors:0603-RES
- B1: value BMP180BREAKOUT -> LDR-ROUND; device mylibrary:BMP180_BREAKOUT -> mylibrary:LDR-ROUND
- moved B1 90.0 mm to (11.5, -7.75), turned to 0 degrees
Connections:
- net +3V3: now also B1.P$1, B2.2; no longer B1.2
- net A0: now also B1.P$2, R6.1
- net GND: now also B2.3, R6.2; no longer B1.3
- net SCL: now also B2.4; no longer B1.4
- net SDA: now also B2.5; no longer B1.5
Changed lines of the file:
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@@
 <element name="R4" library="SparkFun-Resistors" package="0603-RES" value="22R" x="59" y="40.75" rot="R180"/>
 <element name="R5" library="SparkFun-Resistors" package="0603-RES" value="22R" x="59" y="42.25" rot="R180"/>
-<element name="B1" library="mylibrary" package="BMP180_BREAKOUT" value="BMP180BREAKOUT" x="81" y="49.5" rot="R270"/>
+<element name="B2" library="mylibrary" package="BMP180_BREAKOUT" value="BMP180BREAKOUT" x="81" y="49.5" rot="R270"/>
 <element name="D2" library="SparkFun-DiscreteSemi" package="SMA-DIODE" value="MBRA140" x="47.75" y="58.25" rot="R270">
 <attribute name="PROD_ID" value="DIO-08053" x="47.75" y="58.25" size="1.778" layer="27" rot="R270" display="off"/>
@@
 <attribute name="PROD_ID" value="DIO-08053" x="51.25" y="58.25" size="1.778" layer="27" rot="R270" display="off"/>
 </element>
+<element name="B1" library="mylibrary" package="LDR-ROUND" value="LDR-ROUND" x="11.5" y="-7.75"/>
+<element name="R6" library="SparkFun-Resistors" package="0603-RES" value="" x="2.625" y="-16.625"/>
 </elements>
 <signals>
@@
 <contactref element="C9" pad="2"/>
 <contactref element="J1" pad="9"/>
-<contactref element="B1" pad="3"/>
+<contactref element="B2" pad="3"/>
 <polygon width="0.3" layer="1">
 <vertex x="0" y="0"/>
@@
 <vertex x="0" y="80"/>
 </polygon>
-<wire x1="54.25" y1="46.35" x2="54.25" y2="42.25" width="0" layer="19" extent="1-1"/>
-<wire x1="50.25" y1="44.25" x2="51.6" y2="47.25" width="0" layer="19" extent="1-1"/>
-<wire x1="45.75" y1="40.75" x2="42.75" y2="38.4" width="0" layer="19" extent="1-1"/>
-<wire x1="49.75" y1="35.75" x2="49.25" y2="31.15" width="0" layer="19" extent="1-1"/>
+<contactref element="R6" pad="2"/>
+<wire x1="35.968" y1="73.77" x2="48.7" y2="75.85" width="0" layer="19" extent="1-1"/>
+<wire x1="35.968" y1="72.5" x2="35.968" y2="73.77" width="0" layer="19" extent="1-1"/>
+<wire x1="35.968" y1="69.96" x2="35.968" y2="72.5" width="0" layer="19" extent="1-1"/>
+<wire x1="33.05" y1="64.25" x2="35.968" y2="69.96" width="0" layer="19" extent="1-1"/>
+<wire x1="32.5" y1="57.35" x2="33.05" y2="64.25" width="0" layer="19" extent="1-1"/>
+<wire x1="41.45" y1="64.25" x2="35.968" y2="69.96" width="0" layer="19" extent="1-1"/>
+<wire x1="53.85" y1="62" x2="41.45" y2="64.25" width="0" layer="19" extent="1-1"/>
+<wire x1="56.85" y1="62" x2="53.85" y2="62" width="0" layer="19" extent="1-1"/>
+<wire x1="57.25" y1="58.1" x2="56.85" y2="62" width="0" layer="19" extent="1-1"/>
+<wire x1="54.75" y1="54.0501" x2="57.25" y2="58.1" width="0" layer="19" extent="1-1"/>
+<wire x1="57" y1="53.1" x2="54.75" y2="54.0501" width="0" layer="19" extent="1-1"/>
+<wire x1="49.5" y1="54.0501" x2="54.75" y2="54.0501" width="0" layer="19" extent="1-1"/>
+<wire x1="45.525" y1="49.375" x2="49.5" y2="54.0501" width="0" layer="19" extent="1-1"/>
+<wire x1="46.9" y1="47.25" x2="45.525" y2="49.375" width="0" layer="19" extent="1-1"/>
+<wire x1="50.25" y1="44.25" x2="46.9" y2="47.25" width="0" layer="19" extent="1-1"/>
+<wire x1="51.6" y1="47.25" x2="50.25" y2="44.25" width="0" layer="19" extent="1-1"/>
+<wire x1="54.25" y1="46.35" x2="51.6" y2="47.25" width="0" layer="19" extent="1-1"/>
+<wire x1="54.25" y1="42.25" x2="54.25" y2="46.35" width="0" layer="19" extent="1-1"/>
+<wire x1="45.75" y1="40.75" x2="50.25" y2="44.25" width="0" layer="19" extent="1-1"/>
+<wire x1="42.75" y1="38.4" x2="45.75" y2="40.75" width="0" layer="19" extent="1-1"/>
+<wire x1="38.525" y1="39" x2="42.75" y2="38.4" width="0" layer="19" extent="1-1"/>
+<wire x1="38.525" y1="37" x2="38.525" y2="39" width="0" layer="19" extent="1-1"/>
+<wire x1="49.75" y1="35.75" x2="45.75" y2="40.75" width="0" layer="19" extent="1-1"/>
+<wire x1="49.25" y1="31.15" x2="49.75" y2="35.75" width="0" layer="19" extent="1-1"/>
+<wire x1="38.525" y1="46.25" x2="38.525" y2="39" width="0" layer="19" extent="1-1"/>
+<wire x1="82.27" y1="41.88" x2="57" y2="53.1" width="0" layer="19" extent="1-1"/>
+<wire x1="3.475" y1="-16.625" x2="38.525" y2="37" width="0" layer="19" extent="1-1"/>
 </signal>
 <signal name="SWDIO">
@@
 <contactref element="C2" pad="1"/>
 <contactref element="C9" pad="1"/>
-<contactref element="B1" pad="2"/>
+<contactref element="B2" pad="2"/>
 <contactref element="U1" pad="36"/>
 <contactref element="C8" pad="1"/>
@@
 <wire x1="49.25" y1="43.25" x2="49.75" y2="42.75" width="0.3" layer="1"/>
 <wire x1="49.75" y1="42.75" x2="54.25" y2="42.75" width="0.3" layer="1"/>
+<contactref element="B1" pad="P$1"/>
 <wire x1="54.25" y1="44.65" x2="82.27" y2="44.42" width="0" layer="19" extent="1-1"/>
 <wire x1="35.968" y1="75.04" x2="48.55" y2="51.4499" width="0" layer="19" extent="1-1"/>
+<wire x1="6.42" y1="-7.75" x2="40.225" y2="37" width="0" layer="19" extent="1-1"/>
 </signal>
 <signal name="SWCLK">
@@
 <signal name="A0">
 <contactref element="U1" pad="3"/>
+<contactref element="R6" pad="1"/>
+<contactref element="B1" pad="P$2"/>
+<wire x1="16.58" y1="-7.75" x2="45.75" y2="41.75" width="0" layer="19" extent="1-1"/>
+<wire x1="1.775" y1="-16.625" x2="16.58" y2="-7.75" width="0" layer="19" extent="1-1"/>
 </signal>
 <signal name="AREF">
@@
 <signal name="SDA">
 <contactref element="U1" pad="31"/>
-<contactref element="B1" pad="5"/>
+<contactref element="B2" pad="5"/>
 <wire x1="54.25" y1="40.25" x2="82.27" y2="36.8" width="0" layer="19" extent="1-1"/>
 </signal>
 <signal name="SCL">
 <contactref element="U1" pad="32"/>
-<contactref element="B1" pad="4"/>
+<contactref element="B2" pad="4"/>
 <wire x1="54.25" y1="40.75" x2="82.27" y2="39.34" width="0" layer="19" extent="1-1"/>
 </signal>

Commit message: Finished initial version of PCB pending review
Parts:
- added JP1: (no value), pinhead:1X01
- added R7: 4k7, SparkFun-Resistors:0603-RES
- added U$1: RN2483, mylibrary:RN2483
- added U$2: DHT11, mylibrary:DHT11
- moved B2 58.9 mm to (28.4, 23.0)
- moved S1 50.2 mm to (53.5, 14.5), turned to 90 degrees
- moved J1 40.9 mm to (12.1, 40.9)
- moved R6 40.2 mm to (2.62, 23.6), turned to 90 degrees
- moved R1 39.0 mm to (47.9, 18.8), turned to 0 degrees
- moved J2 31.3 mm to (37.9, 48.2)
- moved C8 30.7 mm to (20.5, 21.1), turned to 180 degrees
- moved C1 30.1 mm to (19.9, 36.0)
- moved C10 30.1 mm to (29.4, 46.0)
- moved C11 30.1 mm to (25.1, 50.8)
- moved C12 30.1 mm to (28.1, 50.8)
- moved C13 30.1 mm to (18.5, 38.1)
- moved C2 30.1 mm to (11.5, 25.8)
- moved C3 30.1 mm to (22.9, 36.0)
- moved C4 30.1 mm to (14.9, 28.0)
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Connections:
- new net N$11: JP1.1, U$1.P$23
- net +3V3: now also R7.1, U$1.P$12, U$1.P$34, U$2.P$1
- net D4: now also R7.2, U$2.P$2
- net GND: now also U$1.P$1, U$1.P$11, U$1.P$20, U$1.P$21, U$1.P$22, U$1.P$24, U$1.P$26, U$1.P$27, U$1.P$28, U$1.P$33, U$1.P$41, U$1.P$47, U$1.P$8, U$2.P$4
- net RXD: now also U$1.P$6
- net TXD: now also U$1.P$7
Routing:
- net +3V3: track 44.3 -> 138.0 mm, vias 0 -> 3
- net RESET: track 0.00 -> 50.7 mm, vias 0 -> 4
- net A0: track 0.00 -> 25.7 mm, vias 0 -> 2
- net TXD: track 0.00 -> 24.6 mm, vias 0 -> 2
- net RXD: track 0.00 -> 23.9 mm, vias 0 -> 2
- net N$9: track 0.00 -> 22.0 mm, vias 0 -> 2
- net SDA: track 0.00 -> 20.7 mm
- net SCL: track 0.00 -> 20.3 mm
- net N$4: track 0.00 -> 19.9 mm, vias 0 -> 2
- net V_USB: track 1.77 -> 21.0 mm, vias 0 -> 2
- net SWDIO: track 0.00 -> 18.3 mm
- net D4: track 0.00 -> 14.6 mm
- net SWCLK: track 0.00 -> 14.3 mm
- net N$2: track 0.00 -> 10.9 mm
- net N$11: track 0.00 -> 2.23 mm
- added copper zone on layer 16, net GND
Other:
- board size 100 x 80 mm -> 64.9 x 52.4 mm
