File: Arduino/schematic/mainboard/scrump.sch (EAGLE design)
At the start: 29 parts, among them J1 PINHEAD-FTSH, J2 USB-CON-5PIN-105017-0001, U1 ATSAMD21G-A, U2 LM3671, U3 MCP73831, Y1 32.768kHz

Commit message: Initial PCB
Parts:
- added D3: MBRA140, SparkFun-DiscreteSemi:MBRA140
- added D4: RED 1.8V, SparkFun-LED:LED-RED0603
- C12: value 10uF -> 4.7uF
- C13: value 0.1uF -> 10uF
- C5: value 0.1uF -> 22pF
- C7: value 22pF -> 0.1uF; device SparkFun-Capacitors:CAP0603-CAP -> SparkFun-Capacitors:0.1UF-25V(+80/-20%)(0603)
- C8: device SparkFun-Capacitors:0.1UF-25V(+80/-20%)(0603) -> SparkFun-Capacitors:CAP0603-CAP
- C9: value 4.7uF -> 0.1uF
- D2: value RED 1.8V -> MBRA140; device SparkFun-LED:LED-RED0603 -> SparkFun-DiscreteSemi:MBRA140
- L1: value 2.2uF -> 2.2uH
- R1: value 22R -> 330R
- R2: value 330R -> 1.5k
- R3: value 1.5k -> 5k
- R4: value 2k -> 22R
Connections:
- net PA02 renamed A0
- net PA03 renamed AREF
- net PA04 renamed A3
- net PA05 renamed A4
- net PA06 renamed D8
- net PA07 renamed D9
- net PA08 renamed D4
- net PA09 renamed D3
- net PA10 renamed D1
- net PA11 renamed D0
- net PA12 renamed MISO
- net PA14 renamed D2
- net PA15 renamed D5
- net PA16 renamed D11
- net PA17 renamed D13
- net PA18 renamed D10
- net PA19 renamed D12
- net PA20 renamed D6
- net PA21 renamed D7
- net PB02 renamed A5
- net PB08 renamed A1
- net PB09 renamed A2
- net PB10 renamed MOSI
- net PB11 renamed SCK
- net PB22 renamed TXD
- net PB23 renamed RXD
- removed net +5V: C11.1, D1.A, J2.VBUS
- removed net PA00: C6.1, U1.PA00(XIN32/SER1:0/TC2:0), Y1.1
- removed net PA01: C7.1, U1.PA01(XOUT32/SER1:1/TC2:1), Y1.3
- removed net VCC: C10.1, U2.EN, U2.VIN, U3.VBAT
- new net N$10: D2.C, D3.C, U2.EN, U2.VIN
- new net V_BATT: C11.1, D3.A, U3.VBAT
- new net V_USB: C12.1, D1.A, D2.A, J2.VBUS
- new net XIN32: C5.1, U1.PA00(XIN32/SER1:0/TC2:0), Y1.1
- new net XOUT32: C6.1, U1.PA01(XOUT32/SER1:1/TC2:1), Y1.3
- net +3V3: now also C8.1, C9.1; no longer C12.1, C5.1
- net D-: now also R4.2; no longer R1.2
- net GND: now also R3.1; no longer R4.1
- net N$2: now also R1.2; no longer R2.2
- net N$3: now also C10.1, R2.2; no longer C9.1, R3.2
- net N$6: now also D4.C; no longer D2.C
- net N$7: now also D4.A, R2.1; no longer D2.A, R3.1
- net N$8: now also R3.2; no longer R4.2
- net N$9: now also R4.1; no longer R1.1
- net RESET: now also C7.1, R1.1; no longer C8.1, R2.1
Other:
- moved on the sheet: C1, C10, C11, C12, C13, C2, C3, C4, C5, C6, C7, C8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

Commit message: Added LDR
Parts:
- added B2: BMP180BREAKOUT, mylibrary:BMP180BREAKOUT
- added R6: (no value), SparkFun-Resistors:RESISTOR0603
- B1: value BMP180BREAKOUT -> LDR-ROUND; device mylibrary:BMP180BREAKOUT -> mylibrary:LDR-ROUND
Connections:
- net +3V3: now also B1.1, B2.3V3; no longer B1.3V3
- net A0: now also B1.2, R6.1
- net GND: now also B2.GND, R6.2; no longer B1.GND
- net SCL: now also B2.SCL; no longer B1.SCL
- net SDA: now also B2.SDA; no longer B1.SDA
Changed lines of the file:
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@@
 <part name="R4" library="SparkFun-Resistors" deviceset="RESISTOR" device="0603" value="22R"/>
 <part name="R5" library="SparkFun-Resistors" deviceset="RESISTOR" device="0603" value="22R"/>
-<part name="B1" library="mylibrary" deviceset="BMP180" device="BREAKOUT"/>
+<part name="B2" library="mylibrary" deviceset="BMP180" device="BREAKOUT"/>
 <part name="FRAME2" library="SparkFun-Aesthetics" deviceset="FRAME-A4L" device=""/>
 <part name="+3V36" library="supply1" deviceset="+3V3" device=""/>
@@
 <part name="SUPPLY5" library="SparkFun-Aesthetics" deviceset="V_USB" device=""/>
 <part name="SUPPLY6" library="SparkFun-Aesthetics" deviceset="V_USB" device=""/>
+<part name="B1" library="mylibrary" deviceset="LDR-ROUND" device=""/>
+<part name="R6" library="SparkFun-Resistors" deviceset="RESISTOR" device="0603"/>
+<part name="+3V37" library="supply1" deviceset="+3V3" device=""/>
+<part name="GND20" library="supply1" deviceset="GND" device=""/>
 </parts>
 <sheets>
@@
 </plain>
 <instances>
-<instance part="B1" gate="G$1" x="45.72" y="149.86"/>
+<instance part="B2" gate="G$1" x="45.72" y="149.86"/>
 <instance part="FRAME2" gate="G$1" x="2.54" y="2.54"/>
 <instance part="+3V36" gate="G$1" x="25.4" y="165.1"/>
 <instance part="GND19" gate="1" x="25.4" y="152.4"/>
+<instance part="B1" gate="G$1" x="33.02" y="129.54"/>
+<instance part="R6" gate="G$1" x="40.64" y="121.92" rot="R270"/>
+<instance part="+3V37" gate="G$1" x="25.4" y="134.62"/>
+<instance part="GND20" gate="1" x="40.64" y="111.76"/>
 </instances>
 <busses>
@@
 <net name="+3V3" class="0">
 <segment>
-<pinref part="B1" gate="G$1" pin="3V3"/>
+<pinref part="B2" gate="G$1" pin="3V3"/>
 <pinref part="+3V36" gate="G$1" pin="+3V3"/>
 <wire x1="43.18" y1="160.02" x2="25.4" y2="160.02" width="0.1524" layer="91"/>
 <wire x1="25.4" y1="160.02" x2="25.4" y2="162.56" width="0.1524" layer="91"/>
 </segment>
+<segment>
+<pinref part="+3V37" gate="G$1" pin="+3V3"/>
+<wire x1="25.4" y1="129.54" x2="25.4" y2="132.08" width="0.1524" layer="91"/>
+<pinref part="B1" gate="G$1" pin="1"/>
+<wire x1="25.4" y1="129.54" x2="27.94" y2="129.54" width="0.1524" layer="91"/>
+</segment>
 </net>
 <net name="GND" class="0">
 <segment>
-<pinref part="B1" gate="G$1" pin="GND"/>
+<pinref part="B2" gate="G$1" pin="GND"/>
 <pinref part="GND19" gate="1" pin="GND"/>
 <wire x1="43.18" y1="157.48" x2="25.4" y2="157.48" width="0.1524" layer="91"/>
 <wire x1="25.4" y1="157.48" x2="25.4" y2="154.94" width="0.1524" layer="91"/>
 </segment>
+<segment>
+<pinref part="GND20" gate="1" pin="GND"/>
+<pinref part="R6" gate="G$1" pin="2"/>
+<wire x1="40.64" y1="114.3" x2="40.64" y2="116.84" width="0.1524" layer="91"/>
+</segment>
 </net>
 <net name="SCL" class="0">
 <segment>
-<pinref part="B1" gate="G$1" pin="SCL"/>
+<pinref part="B2" gate="G$1" pin="SCL"/>
 <wire x1="43.18" y1="154.94" x2="38.1" y2="154.94" width="0.1524" layer="91"/>
 <label x="38.1" y="154.94" size="1.27" layer="95" rot="R180" xref="yes"/>
@@
 <net name="SDA" class="0">
 <segment>
-<pinref part="B1" gate="G$1" pin="SDA"/>
+<pinref part="B2" gate="G$1" pin="SDA"/>
 <wire x1="43.18" y1="152.4" x2="38.1" y2="152.4" width="0.1524" layer="91"/>
 <label x="38.1" y="152.4" size="1.27" layer="95" rot="R180" xref="yes"/>
 </segment>
 </net>
+<net name="A0" class="0">
+<segment>
+<pinref part="R6" gate="G$1" pin="1"/>
+<pinref part="B1" gate="G$1" pin="2"/>
+<wire x1="40.64" y1="127" x2="40.64" y2="129.54" width="0.1524" layer="91"/>
+<wire x1="40.64" y1="129.54" x2="38.1" y2="129.54" width="0.1524" layer="91"/>
+<wire x1="40.64" y1="129.54" x2="43.18" y2="129.54" width="0.1524" layer="91"/>
+<junction x="40.64" y="129.54"/>
+<label x="43.18" y="129.54" size="1.27" layer="95" font="vector" xref="yes"/>
+</segment>
+</net>

Commit message: Finished initial version of PCB pending review
Parts:
- added JP1: (no value), pinhead:PINHD-1X1
- added R7: 4k7, SparkFun-Resistors:RESISTOR0603
- added U$1: RN2483, mylibrary:RN2483
- added U$2: DHT11, mylibrary:DHT11
Connections:
- new net N$11: JP1.1, U$1.RFH
- net +3V3: now also R7.1, U$1.VCC, U$2.VCC
- net D4: now also R7.2, U$2.DATA
- net GND: now also U$1.GND, U$2.GND
- net RXD: now also U$1.TX
- net TXD: now also U$1.RX
Changed lines of the file:
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@@
 <part name="+3V37" library="supply1" deviceset="+3V3" device=""/>
 <part name="GND20" library="supply1" deviceset="GND" device=""/>
+<part name="U$1" library="mylibrary" deviceset="RN2483" device=""/>
+<part name="+3V1" library="supply1" deviceset="+3V3" device=""/>
+<part name="GND21" library="supply1" deviceset="GND" device=""/>
+<part name="U$2" library="mylibrary" deviceset="DHT11" device=""/>
+<part name="+3V2" library="supply1" deviceset="+3V3" device=""/>
+<part name="GND22" library="supply1" deviceset="GND" device=""/>
+<part name="R7" library="SparkFun-Resistors" deviceset="RESISTOR" device="0603" value="4k7"/>
+<part name="+3V3" library="supply1" deviceset="+3V3" device=""/>
+<part name="JP1" library="pinhead" deviceset="PINHD-1X1" device=""/>
 </parts>
 <sheets>
@@
 <instance part="SUPPLY5" gate="G$1" x="254" y="53.34"/>
 <instance part="SUPPLY6" gate="G$1" x="256.54" y="147.32"/>
+<instance part="U$1" gate="G$1" x="50.8" y="25.4"/>
+<instance part="+3V1" gate="G$1" x="43.18" y="43.18"/>
+<instance part="GND21" gate="1" x="43.18" y="22.86"/>
+<instance part="JP1" gate="G$1" x="25.4" y="30.48" rot="R180"/>
 </instances>
 <busses>
@@
 <label x="228.6" y="165.1" size="1.778" layer="95"/>
 </segment>
+<segment>
+<pinref part="U$1" gate="G$1" pin="GND"/>
+<pinref part="GND21" gate="1" pin="GND"/>
+<wire x1="45.72" y1="27.94" x2="43.18" y2="27.94" width="0.1524" layer="91"/>
+<wire x1="43.18" y1="27.94" x2="43.18" y2="25.4" width="0.1524" layer="91"/>
+</segment>
 </net>
 <net name="SWDIO" class="0">
@@
 <junction x="33.02" y="147.32"/>
 </segment>
+<segment>
+<pinref part="+3V1" gate="G$1" pin="+3V3"/>
+<wire x1="43.18" y1="38.1" x2="43.18" y2="40.64" width="0.1524" layer="91"/>
+<pinref part="U$1" gate="G$1" pin="VCC"/>
+<wire x1="43.18" y1="38.1" x2="45.72" y2="38.1" width="0.1524" layer="91"/>
+</segment>
 </net>
 <net name="SWCLK" class="0">
@@
 <label x="116.84" y="99.06" size="1.27" layer="95" xref="yes"/>
 </segment>
+<segment>
+<pinref part="U$1" gate="G$1" pin="RX"/>
+<wire x1="45.72" y1="35.56" x2="40.64" y2="35.56" width="0.1524" layer="91"/>
+<label x="40.64" y="35.56" size="1.27" layer="95" rot="R180" xref="yes"/>
+</segment>
 </net>
 <net name="RXD" class="0">
@@
 <wire x1="109.22" y1="96.52" x2="116.84" y2="96.52" width="0.1524" layer="91"/>
 <label x="116.84" y="96.52" size="1.27" layer="95" xref="yes"/>
+</segment>
+<segment>
+<pinref part="U$1" gate="G$1" pin="TX"/>
+<wire x1="45.72" y1="33.02" x2="40.64" y2="33.02" width="0.1524" layer="91"/>
+<label x="40.64" y="33.02" size="1.27" layer="95" rot="R180" xref="yes"/>
 </segment>
 </net>
@@
 <wire x1="177.8" y1="50.8" x2="177.8" y2="60.96" width="0.1524" layer="91"/>
 <wire x1="177.8" y1="60.96" x2="172.72" y2="60.96" width="0.1524" layer="91"/>
+</segment>
+</net>
+<net name="N$11" class="0">
+<segment>
+<pinref part="U$1" gate="G$1" pin="RFH"/>
+<pinref part="JP1" gate="G$1" pin="1"/>
+<wire x1="45.72" y1="30.48" x2="27.94" y2="30.48" width="0.1524" layer="91"/>
 </segment>
 </net>
@@
 <instance part="+3V37" gate="G$1" x="25.4" y="134.62"/>
 <instance part="GND20" gate="1" x="40.64" y="111.76"/>
+<instance part="U$2" gate="G$1" x="106.68" y="152.4"/>
+<instance part="+3V2" gate="G$1" x="99.06" y="175.26"/>
+<instance part="GND22" gate="1" x="99.06" y="149.86"/>
+<instance part="R7" gate="G$1" x="91.44" y="165.1" rot="R270"/>
+<instance part="+3V3" gate="G$1" x="91.44" y="175.26"/>
 </instances>
 <busses>
@@
 <wire x1="25.4" y1="129.54" x2="27.94" y2="129.54" width="0.1524" layer="91"/>
 </segment>
+<segment>
+<pinref part="U$2" gate="G$1" pin="VCC"/>
+<pinref part="+3V2" gate="G$1" pin="+3V3"/>
+<wire x1="101.6" y1="160.02" x2="99.06" y2="160.02" width="0.1524" layer="91"/>
+<wire x1="99.06" y1="160.02" x2="99.06" y2="172.72" width="0.1524" layer="91"/>
+</segment>
+<segment>
+<pinref part="R7" gate="G$1" pin="1"/>
+<pinref part="+3V3" gate="G$1" pin="+3V3"/>
+<wire x1="91.44" y1="170.18" x2="91.44" y2="172.72" width="0.1524" layer="91"/>
+</segment>
 </net>
 <net name="GND" class="0">
@@
 <pinref part="R6" gate="G$1" pin="2"/>
 <wire x1="40.64" y1="114.3" x2="40.64" y2="116.84" width="0.1524" layer="91"/>
+</segment>
+<segment>
+<pinref part="U$2" gate="G$1" pin="GND"/>
+<pinref part="GND22" gate="1" pin="GND"/>
+<wire x1="101.6" y1="154.94" x2="99.06" y2="154.94" width="0.1524" layer="91"/>
+<wire x1="99.06" y1="154.94" x2="99.06" y2="152.4" width="0.1524" layer="91"/>
 </segment>
 </net>
@@
 </segment>
 </net>
+<net name="D4" class="0">
+<segment>
+<pinref part="U$2" gate="G$1" pin="DATA"/>
+<pinref part="R7" gate="G$1" pin="2"/>
+<wire x1="101.6" y1="157.48" x2="91.44" y2="157.48" width="0.1524" layer="91"/>
+<wire x1="91.44" y1="157.48" x2="91.44" y2="160.02" width="0.1524" layer="91"/>
+<wire x1="91.44" y1="157.48" x2="88.9" y2="157.48" width="0.1524" layer="91"/>
+<junction x="91.44" y="157.48"/>
+<label x="88.9" y="157.48" size="1.778" layer="95" rot="R180" xref="yes"/>
+</segment>
+</net>
